File: cubesat Sim board.kicad_pcb (KiCad board)
At the start: 2 copper layers, 80.2 x 80.2 mm, 41 parts, among them J1 HASP Power In, J10 USB_2_OUT, J2 PI Bus, J3 JST_Solar, J4 JST_Main(optional), J5 INA219, J6 HASP Data In, J7 USB_IN, J8 USB_2, J9 USB_1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

Commit message: Fixes to some ERC checks. Tracking down a potential short issue.
Parts:
- removed ? (x3): , 
- removed REF**: MountingHole_2.7mm_M2.5_Pad, MountingHole:MountingHole_2.7mm_M2.5_Pad
- J4: value JST_Main(optional) -> 5V TP
- moved J4 58.9 mm to (149.7, 108.1)
Connections:
- net /28V renamed 28V
- net /EN renamed EN
- net /SCL renamed SCL
- net /SDA renamed SDA
- net /SW renamed Net-(U1-SW)
- C10 pad 2: /BATT_SW -> VCC
- C11 pad 2: /BATT_SW -> VCC
- C14 pad 2: /BATT_SW -> VCC
- C5 pad 2: /4v6 -> 5V
- J2 pad 1: /PI_3V3 -> unconnected-(J2-Pin_1-Pad1)
- J2 pad 2: /BATT_SW -> VCC
- J2 pad 4: /BATT_SW -> VCC
- J4 pad 1: /BATT_SW -> GND
- J4 pad 2: GND -> 5V
- J5 pad VCC: /BATT_SW -> VCC
- J5 pad Vin+: /4v6 -> 5V
- J5 pad Vin-: /BATT_SW -> VCC
- L1 pad 2: /4v6 -> 5V
- R2 pad 1: /4v6 -> 5V
- R6 pad 1: /BATT_SW -> VCC
- R7 pad 1: /BATT_SW -> VCC
- U2 pad 16: /BATT_SW -> VCC
- U3 pad 20: /BATT_SW -> VCC
- U3 pad 4: /BATT_SW -> VCC
Routing:
- net 5V: track 0.00 -> 10.6 mm
- net /4v6: track 10.4 -> 0.00 mm
- net VCC: track 0.00 -> 2.42 mm
- net /BATT_SW: track 2.42 -> 0.00 mm
- added copper zone on F.Cu, net 5V
- added copper zone on F.Cu, net VCC
- removed copper zone on F.Cu, net /4v6
- removed copper zone on F.Cu, net /BATT_SW
